File: Adafruit-Feather.brd (EAGLE design)
At the start: 50.8 x 22.9 mm, 40 parts, among them IC1 CP2104, Q1 mmbt2222, Q2 mmbt2222, Q3 DMG3415U, SW2 KMR2, U2 AP2112-3.3, U3 MCP73831T-2ACI/OT, X1 JSTPH, X2 ESP32_WROOM32_SKINNY, X4 20329

Commit message: Huzzah #2
Connections:
- removed net A3_I39: JP1.9, X2.5
- removed net A4_IO36: JP1.8, X2.4
- removed net N$12: Q1.1, R13.5
- new net S$1: Q1.3, R13.6
- new net S$10: X2.10
- new net S$2: CHG.A
- new net S$3: X4.VBUS
- new net S$4: IC1.8, U3.4
- new net S$5: Q3.1
- new net S$6: JP1.10
- new net S$7: JP1.12
- new net S$8: X2.5
- new net S$9: X2.4
- net A0_DAC2: no longer JP1.12
- net A1_DAC1: no longer X2.10
- net A2_I34: no longer JP1.10
- net RESET: no longer Q1.3, R13.6
- net VBUS: no longer CHG.A, IC1.8, Q3.1, U3.4, X4.VBUS
Routing:
- net VBUS: track 56.2 -> 14.1 mm, vias 4 -> 1
- net A0_DAC2: track 32.4 -> 2.31 mm
- net A3_I39: track 28.8 -> 0.00 mm, vias 1 -> 0
- net A2_I34: track 31.8 -> 8.23 mm, vias 2 -> 1
- net S$4: track 0.00 -> 21.0 mm, vias 0 -> 3
- net A4_IO36: track 20.0 -> 0.00 mm, vias 1 -> 0
- net A1_DAC1: track 25.0 -> 8.63 mm, vias 1 -> 0
- net S$7: track 0.00 -> 10.7 mm
- net S$9: track 0.00 -> 7.92 mm, vias 0 -> 1
- net S$6: track 0.00 -> 7.64 mm, vias 0 -> 1
- net S$8: track 0.00 -> 7.17 mm, vias 0 -> 1
- net N$12: track 3.32 -> 0.00 mm
- net RESET: track 48.1 -> 45.7 mm
- net S$10: track 0.00 -> 1.97 mm, vias 0 -> 1
- net S$1: track 0.00 -> 1.24 mm

Commit message: Huzzah #3
Parts:
- removed JP1: (no value), microbuilder:1X16_ROUND_MIN
- removed U$31: MOUNTINGHOLE2.5, microbuilder:MOUNTINGHOLE_2.5_PLATED
Connections:
- net S$8 renamed A3_I39
- net S$9 renamed A4_IO36
- removed net S$10: X2.10
- removed net S$3: X4.VBUS
- removed net S$4: IC1.8, U3.4
- removed net S$5: Q3.1
- removed net S$6: JP1.10
- removed net S$7: JP1.12
- new net N$12: Q1.1, R13.5
- net 3.3V: no longer JP1.15
- net A1_DAC1: now also X2.10; no longer JP1.11
- net A5_IO4: no longer JP1.7
- net GND: no longer JP1.13
- net IO15_A8: no longer X2.23
- net IO16: no longer JP1.3
- net IO17: no longer JP1.2
- net IO21: no longer JP1.1
- net MISO: no longer JP1.4
- net MOSI: no longer JP1.5
- net RESET: now also Q1.3, R13.6; no longer JP1.16
- net S$1: now also C3.1, JP3.1, X1.2; no longer Q1.3, R13.6
- net S$2: now also X2.23; no longer CHG.A
- net SCK: no longer JP1.6
- net VBAT: no longer C3.1, JP3.1, X1.2
- net VBUS: now also CHG.A, IC1.8, Q3.1, U3.4, X4.VBUS
Routing:
- net VBUS: track 14.1 -> 56.2 mm, vias 1 -> 4
- net A0_DAC2: track 2.31 -> 32.4 mm
- net A2_I34: track 8.23 -> 31.8 mm, vias 1 -> 2
- net A3_I39: track 7.17 -> 28.8 mm
- net S$4: track 21.0 -> 0.00 mm, vias 3 -> 0
- net A1_DAC1: track 8.63 -> 25.0 mm, vias 0 -> 1
- net VBAT: track 28.4 -> 13.9 mm
- net A4_IO36: track 7.92 -> 20.0 mm
- net S$7: track 10.7 -> 0.00 mm
- net S$1: track 1.24 -> 10.1 mm
- net S$6: track 7.64 -> 0.00 mm, vias 1 -> 0
- net N$12: track 0.00 -> 3.32 mm
- net RESET: track 45.7 -> 48.1 mm
- net S$10: track 1.97 -> 0.00 mm, vias 1 -> 0
- net IO15_A8: track 14.7 -> 14.1 mm
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
Commit message: Huzzah #3
Connections:
- removed net S$1: C3.1, JP3.1, X1.2
- removed net S$2: X2.23
- net IO15_A8: now also X2.23
- net VBAT: now also C3.1, JP3.1, X1.2
Routing:
- net VBAT: track 13.9 -> 28.4 mm
- net S$1: track 10.1 -> 0.00 mm
- net IO15_A8: track 14.1 -> 14.7 mm
- net S$2: track 0.62 -> 0.00 mm
- net GND: vias 51 -> 47

Commit message: Huzzah #3
Parts:
- removed C2: 10uF, microbuilder:0805-NO
- removed IC1: CP2104, microbuilder:QFN24_4MM_SMSC
- removed R1, R3: 100K, microbuilder:0603-NO
- removed R4: 4.7K, microbuilder:0603-NO
- added E$1: (no value), allegro:PLCC44
- added JP1: (no value), microbuilder:1X16_ROUND_MIN
- added U$31: MOUNTINGHOLE2.5, microbuilder:MOUNTINGHOLE_2.5_PLATED
Connections:
- new net S$1: X2.10
- net 3.3V: now also JP1.15; no longer C2.1, IC1.5, IC1.6, IC1.7
- net A0_DAC2: now also JP1.12
- net A13_I35: no longer R1.1, R3.2
- net A1_DAC1: now also JP1.11; no longer X2.10
- net A2_I34: now also JP1.10
- net A3_I39: now also JP1.9
- net A4_IO36: now also JP1.8
- net A5_IO4: now also JP1.7
- net DTR: no longer IC1.23
- net GND: now also JP1.13; no longer C2.2, IC1.2, IC1.THERM, R3.1, R4.1
- net IO16: now also JP1.3
- net IO17: now also JP1.2
- net IO21: now also JP1.1
- net MISO: now also JP1.4
- net MOSI: now also JP1.5
- net N$2: no longer IC1.3
- net N$4: no longer R4.2
- net N$6: no longer IC1.4
- net RESET: now also JP1.16
- net RTS: no longer IC1.19
- net RXD0: no longer IC1.21
- net SCK: now also JP1.6
- net TXD0: no longer IC1.20
- net VBAT: no longer R1.2
- net VBUS: no longer IC1.8
Routing:
- net A1_DAC1: track 25.0 -> 11.9 mm, vias 1 -> 0
- net S$1: track 0.00 -> 6.63 mm, vias 0 -> 1
- net GND: vias 47 -> 56
Other:
- board size 50.8 x 22.9 mm -> 58.9 x 45.4 mm
