File: Adafruit-Feather.sch (EAGLE design)
At the start: 34 parts, among them IC1 CP2104, Q1 mmbt2222, Q2 mmbt2222, Q3 DMG3415U, SW2 KMR2, U2 AP2112-3.3, U3 MCP73831T-2ACI/OT, X1 JSTPH, X2 ESP32_WROOM32_SKINNY, X4 20329

Commit message: changes
Parts:
- removed C1: 10uF, microbuilder:CAP_CERAMIC0805-NOOUTLINE
- removed C4: 1uF, microbuilder:CAP_CERAMIC0603_NO
- removed Q3: DMG3415U, microbuilder:MOSFET-P
- removed R12: 100K, microbuilder:RESISTOR_0603_NOOUT
- removed R13: 10K, microbuilder:RESISTOR_4PACK
- added R11: 1K, microbuilder:RESISTOR_0603MP
- added R5: 10K, microbuilder:RESISTOR_0603MP
- added R6: 4.7K, microbuilder:RESISTOR_0603_NOOUT
- added R8: 10K\, microbuilder:RESISTOR_0603_NOOUT
- added R9: 10K, microbuilder:RESISTOR_0603_NOOUT
- added SJ1: (no value), microbuilder:SOLDERJUMPER_CLOSED
- JP1: device microbuilder:HEADER-1X16_MIN -> microbuilder:HEADER-1X16ROUND
- JP3: device microbuilder:HEADER-1X12_MIN -> microbuilder:HEADER-1X12
- R1, R3, R7: value 100K -> 10K
- R4: value 4.7K -> 10K
- U$34, U$35: value FIDUCIAL_1MM -> FIDUCIAL""; device microbuilder:FIDUCIAL_1MM -> microbuilder:FIDUCIAL""
- U2: value AP2112-3.3 -> SPX3819
- X2: value ESP32_WROOM32_SKINNY -> ESP-12; device microbuilder:ESP32_WROOM32_SKINNY -> microbuilder:ESP-12E
Connections:
- removed net A0_DAC2: JP1.12, X2.IO26/DAC2/A2_9
- removed net A13_I35: R1.1, R3.2, X2.I35/A1_7
- removed net A1_DAC1: JP1.11, X2.IO25/DAC1/A2_8
- removed net A2_I34: JP1.10, X2.I34/A1_6
- removed net A3_I39: JP1.9, X2.IO39/SEN_VN/A1_3
- removed net A4_IO36: JP1.8, X2.IO36/SEN_VP/A1_0
- removed net A5_IO4: JP1.7, X2.IO4/A2_0
- removed net IO12_A11: JP3.5, X2.IO12/A2_5
- removed net IO13_A12: JP3.4, R10.1, X2.IO13/A2_4
- removed net IO14_A6: JP3.10, X2.IO14/A2_6
- removed net IO15_A8: JP3.8, X2.IO15/A2_3
- removed net IO16: JP1.3, X2.IO16
- removed net IO17: JP1.2, X2.IO17
- removed net IO21: JP1.1, X2.IO21
- removed net IO27_A10: JP3.6, X2.IO27/A2_7
- removed net IO32_A7: JP3.9, X2.IO32/A1_4/X32P
- removed net IO33_A9: JP3.7, X2.IO33/A1_5/X32N
- removed net MISO: JP1.4, X2.IO19
- removed net MOSI: JP1.5, X2.IO18
- removed net RXD0: IC1G$1.TXD, X2.RXD0
- removed net SCK: JP1.6, X2.IO5
- removed net SCL: JP3.11, X2.IO22
- removed net SDA: JP3.12, X2.IO23
- removed net TXD0: IC1G$1.RXD, X2.TXD0
- new net ADC: JP1.12, X2.ADC
- new net CH_PD: JP1.1, R1.1, X2.CH_PD
- new net GPIO12/MISO: JP1.4, JP3.5, X2.GPIO12
- new net GPIO13/MOSI: JP1.5, JP3.6, X2.GPIO13
- new net GPIO14/SCK: JP1.6, JP3.4, X2.GPIO14
- new net GPIO15: JP3.7, R6.2, X2.GPIO15
- new net GPIO16: JP3.9, X2.GPIO16
- new net GPIO4/SDA: JP3.12, X2.GPIO4
- new net GPIO5/SCL: JP3.11, X2.GPIO5
- new net RXD: JP1.3, R11.2, X2.RXD
- new net TXD: IC1G$1.RXD, JP1.2, X2.TXD
- new net USB_RX: IC1G$1.TXD, R11.1
- net 3.3V: now also D3.A, R1.2, R3.2, R9.2, X2.VCC; no longer C1.1, R13G$3.1, X2.3.3V
- net DTR: now also R4.1; no longer R13G$4.1
- net GND: now also R6.1, R8.2; no longer C1.2, C4.2, D3.C, R12.1, R3.1, R4.1
- net GPIO0: now also JP3.8, R10.1, X2.GPIO0; no longer X2.IO0/A2_1
- net GPIO2: now also JP3.10, R9.1, X2.GPIO2; no longer X2.IO2/A2_2
- net N$12: now also R4.2; no longer R13G$4.2
- net N$13: now also R5.2; no longer R13G$2.1
- net N$4: now also R8.1; no longer R4.2
- net N$5: now also D3.C; no longer D3.A
- net N$7: now also SJ1.1, U3.VBAT; no longer C6.1, D4.C, Q3.S, R7.2, U2.IN
- net RESET: now also R3.1, X2.RESET; no longer C4.1, R13G$3.2, X2.EN
- net RTS: now also R5.1; no longer R13G$2.2
- net VBAT: now also D4.A, SJ1.2; no longer Q3.D, R1.2, U3.VBAT
- net VBUS: now also C6.1, D4.C, R7.2, U2.IN; no longer D4.A, Q3.G, R12.2
Other:
- note added: "ESP8266 MODULE + AUTORESET"
- note removed: "ESP3212 MODULE + AUTORESET"
- note removed: "NC: IO0,IO2 VBAT SENSE: IO35 LED: IO13"
- moved on the sheet: C3, C6, C7, C8, CHG, D3, D4, R1, R10, R2, R3, R4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
